File: pcb/weathion-display/esp12.sch (KiCad schematic (older format))
At the start: 12 parts

Commit message: full schematic done
Parts:
- C1, C2, C3, C4, C5, C6: renamed from C?; footprint (none) -> Capacitors:C_0603
- J7: renamed from J?; footprint (none) -> Connector_Header:PinHeader_1x02_P2.54mm_Vertical
- R3, R4, R5: renamed from R?; footprint (none) -> Resistors:R_0603
- gave numbers to parts that had none: 2
Connections:
- net Gas_A0: now reaches U2.2 (ADC)
- net SDA: now reaches U2.6 (GPIO12)
- net SCL: now reaches U2.7 (GPIO13)
Other:
- moved on the sheet: C1, R3, R4, R5
Changed lines of the file:
@@
 P 5000 3150
 AR Path="/5E5B8105" Ref="U?"  Part="1"
-AR Path="/5E5A8A9D/5E5B8105" Ref="U?"  Part="1"
-F 0 "U?" H 5000 4067 50  0000 C CNN
+AR Path="/5E5A8A9D/5E5B8105" Ref="U2"  Part="1"
+F 0 "U2" H 5000 4067 50  0000 C CNN
 F 1 "ESP12" H 5000 3976 50  0000 C CNN
 F 2 "Module:ESP-12E" H 5000 2000 50  0001 C CNN
@@
 L Resistor_0603:R R?
 U 1 1 5E5B810B
-P 4250 2200
+P 4100 2200
 AR Path="/5E5B810B" Ref="R?"  Part="1"
-AR Path="/5E5A8A9D/5E5B810B" Ref="R?"  Part="1"
-F 0 "R?" H 4320 2246 50  0000 L CNN
-F 1 "1k" H 4320 2155 50  0000 L CNN
-F 2 "" V 4180 2200 50  0001 C CNN
-F 3 "~" H 4250 2200 50  0001 C CNN
-	1    4250 2200
+AR Path="/5E5A8A9D/5E5B810B" Ref="R5"  Part="1"
+F 0 "R5" H 4170 2246 50  0000 L CNN
+F 1 "1k" H 4170 2155 50  0000 L CNN
+F 2 "Resistors:R_0603" V 4030 2200 50  0001 C CNN
+F 3 "~" H 4100 2200 50  0001 C CNN
+	1    4100 2200
 	1    0    0    -1
 $EndComp
@@
 L Resistor_0603:R R?
 U 1 1 5E5B8111
-P 4150 3400
+P 3950 3400
 AR Path="/5E5B8111" Ref="R?"  Part="1"
-AR Path="/5E5A8A9D/5E5B8111" Ref="R?"  Part="1"
-F 0 "R?" H 4220 3446 50  0000 L CNN
-F 1 "4.7k" H 4220 3355 50  0000 L CNN
-F 2 "" V 4080 3400 50  0001 C CNN
-F 3 "~" H 4150 3400 50  0001 C CNN
-	1    4150 3400
+AR Path="/5E5A8A9D/5E5B8111" Ref="R4"  Part="1"
+F 0 "R4" H 4020 3446 50  0000 L CNN
+F 1 "4.7k" H 4020 3355 50  0000 L CNN
+F 2 "Resistors:R_0603" V 3880 3400 50  0001 C CNN
+F 3 "~" H 3950 3400 50  0001 C CNN
+	1    3950 3400
 	1    0    0    -1
 $EndComp
@@
 L Power:GND #PWR?
 U 1 1 5E5B8117
-P 4150 3650
+P 3950 3650
 AR Path="/5E5B8117" Ref="#PWR?"  Part="1"
-AR Path="/5E5A8A9D/5E5B8117" Ref="#PWR?"  Part="1"
-F 0 "#PWR?" H 4150 3400 50  0001 C CNN
-F 1 "GND" H 4150 3500 50  0001 C CNN
-F 2 "" H 4150 3650 50  0001 C CNN
-F 3 "~" H 4150 3650 50  0001 C CNN
-	1    4150 3650
+AR Path="/5E5A8A9D/5E5B8117" Ref="#PWR0102"  Part="1"
+F 0 "#PWR0102" H 3950 3400 50  0001 C CNN
+F 1 "GND" H 3950 3500 50  0001 C CNN
+F 2 "" H 3950 3650 50  0001 C CNN
+F 3 "~" H 3950 3650 50  0001 C CNN
+	1    3950 3650
 	1    0    0    -1
 $EndComp
@@
 P 5750 2250
 AR Path="/5E5B811D" Ref="C?"  Part="1"
-AR Path="/5E5A8A9D/5E5B811D" Ref="C?"  Part="1"
-F 0 "C?" H 5868 2296 50  0000 L CNN
+AR Path="/5E5A8A9D/5E5B811D" Ref="C5"  Part="1"
+F 0 "C5" H 5868 2296 50  0000 L CNN
 F 1 "0.1uF" H 5868 2205 50  0000 L CNN
-F 2 "" H 5788 2100 50  0001 C CNN
+F 2 "Capacitors:C_0603" H 5788 2100 50  0001 C CNN
 F 3 "~" H 5750 2250 50  0001 C CNN
 	1    5750 2250
@@
 P 5600 3900
 AR Path="/5E5B8123" Ref="#PWR?"  Part="1"
-AR Path="/5E5A8A9D/5E5B8123" Ref="#PWR?"  Part="1"
-F 0 "#PWR?" H 5600 3650 50  0001 C CNN
+AR Path="/5E5A8A9D/5E5B8123" Ref="#PWR0103"  Part="1"
+F 0 "#PWR0103" H 5600 3650 50  0001 C CNN
 F 1 "GND" H 5600 3750 50  0001 C CNN
 F 2 "" H 5600 3900 50  0001 C CNN
@@
 P 5850 3900
 AR Path="/5E5B8129" Ref="#PWR?"  Part="1"
-AR Path="/5E5A8A9D/5E5B8129" Ref="#PWR?"  Part="1"
-F 0 "#PWR?" H 5850 3650 50  0001 C CNN
+AR Path="/5E5A8A9D/5E5B8129" Ref="#PWR0104"  Part="1"
+F 0 "#PWR0104" H 5850 3650 50  0001 C CNN
 F 1 "GND" H 5850 3750 50  0001 C CNN
 F 2 "" H 5850 3900 50  0001 C CNN
@@
 P 6050 3550
 AR Path="/5E5B812F" Ref="J?"  Part="1"
-AR Path="/5E5A8A9D/5E5B812F" Ref="J?"  Part="1"
-F 0 "J?" H 6130 3592 50  0000 L CNN
+AR Path="/5E5A8A9D/5E5B812F" Ref="J7"  Part="1"
+F 0 "J7" H 6130 3592 50  0000 L CNN
 F 1 "Header_01x02" H 6130 3501 50  0000 L CNN
-F 2 "" H 6050 3400 50  0001 C CNN
+F 2 "Connector_Header:PinHeader_1x02_P2.54mm_Vertical" H 6050 3400 50  0001 C CNN
 F 3 "" H 6050 3400 50  0001 C CNN
 	1    6050 3550
 	1    0    0    -1
 $EndComp
-Text GLabel 3850 1950 0    50   Input ~ 0
+Text GLabel 3700 1950 0    50   Input ~ 0
 3V3
 $Comp
@@
 P 5750 2000
 AR Path="/5E5B8136" Ref="#PWR?"  Part="1"
-AR Path="/5E5A8A9D/5E5B8136" Ref="#PWR?"  Part="1"
-F 0 "#PWR?" H 5750 1750 50  0001 C CNN
+AR Path="/5E5A8A9D/5E5B8136" Ref="#PWR0105"  Part="1"
+F 0 "#PWR0105" H 5750 1750 50  0001 C CNN
 F 1 "GND" H 5750 1850 50  0001 C CNN
 F 2 "" H 5750 2000 50  0001 C CNN
@@
 $EndComp
 Wire Wire Line
-	3850 1950 3900 1950
-Wire Wire Line
-	4250 1950 4250 2050
-Wire Wire Line
-	3900 1950 4250 1950
-Connection ~ 3900 1950
-Wire Wire Line
-	3900 2350 3900 2500
-Wire Wire Line
-	3900 1950 3900 2050
+	3700 1950 3750 1950
+Wire Wire Line
+	4100 1950 4100 2050
+Wire Wire Line
+	3750 1950 4100 1950
+Connection ~ 3750 1950
+Wire Wire Line
+	3750 2350 3750 2500
+Wire Wire Line
+	3750 1950 3750 2050
 $Comp
 L Power:GND #PWR?
 U 1 1 5E5B8142
-P 3900 3000
+P 3750 3000
 AR Path="/5E5B8142" Ref="#PWR?"  Part="1"
-AR Path="/5E5A8A9D/5E5B8142" Ref="#PWR?"  Part="1"
-F 0 "#PWR?" H 3900 2750 50  0001 C CNN
-F 1 "GND" H 3900 2850 50  0001 C CNN
-F 2 "" H 3900 3000 50  0001 C CNN
-F 3 "~" H 3900 3000 50  0001 C CNN
-	1    3900 3000
+AR Path="/5E5A8A9D/5E5B8142" Ref="#PWR0106"  Part="1"
+F 0 "#PWR0106" H 3750 2750 50  0001 C CNN
+F 1 "GND" H 3750 2850 50  0001 C CNN
+F 2 "" H 3750 3000 50  0001 C CNN
+F 3 "~" H 3750 3000 50  0001 C CNN
+	1    3750 3000
 	1    0    0    -1
 $EndComp
@@
 L Capacitor_0603:C C?
 U 1 1 5E5B8148
-P 3900 2750
+P 3750 2750
 AR Path="/5E5B8148" Ref="C?"  Part="1"
-AR Path="/5E5A8A9D/5E5B8148" Ref="C?"  Part="1"
-F 0 "C?" H 4018 2796 50  0000 L CNN
-F 1 "0.1uF" H 4018 2705 50  0000 L CNN
-F 2 "" H 3938 2600 50  0001 C CNN
-F 3 "~" H 3900 2750 50  0001 C CNN
-	1    3900 2750
+AR Path="/5E5A8A9D/5E5B8148" Ref="C1"  Part="1"
+F 0 "C1" H 3868 2796 50  0000 L CNN
+F 1 "0.1uF" H 3868 2705 50  0000 L CNN
+F 2 "Capacitors:C_0603" H 3788 2600 50  0001 C CNN
+F 3 "~" H 3750 2750 50  0001 C CNN
+	1    3750 2750
 	1    0    0    -1
 $EndComp
@@
 L Resistor_0603:R R?
 U 1 1 5E5B814E
-P 3900 2200
+P 3750 2200
 AR Path="/5E5B814E" Ref="R?"  Part="1"
-AR Path="/5E5A8A9D/5E5B814E" Ref="R?"  Part="1"
-F 0 "R?" H 3970 2246 50  0000 L CNN
-F 1 "10k" H 3970 2155 50  0000 L CNN
-F 2 "" V 3830 2200 50  0001 C CNN
-F 3 "~" H 3900 2200 50  0001 C CNN
-	1    3900 2200
-	1    0    0    -1
-$EndComp
-Wire Wire Line
-	4500 2500 3900 2500
-Connection ~ 3900 2500
-Wire Wire Line
-	3900 2500 3900 2600
-Wire Wire Line
-	4250 2350 4250 2700
-Wire Wire Line
-	4250 2700 4500 2700
-Wire Wire Line
-	3900 3000 3900 2900
-Wire Wire Line
-	4500 3000 4150 3000
-Wire Wire Line
-	4150 3000 4150 3250
-Wire Wire Line
-	4150 3550 4150 3650
+AR Path="/5E5A8A9D/5E5B814E" Ref="R3"  Part="1"
+F 0 "R3" H 3820 2246 50  0000 L CNN
+F 1 "10k" H 3820 2155 50  0000 L CNN
+F 2 "Resistors:R_0603" V 3680 2200 50  0001 C CNN
+F 3 "~" H 3750 2200 50  0001 C CNN
+	1    3750 2200
+	1    0    0    -1
+$EndComp
+Wire Wire Line
+	4500 2500 3750 2500
+Connection ~ 3750 2500
+Wire Wire Line
+	3750 2500 3750 2600
+Wire Wire Line
+	4100 2350 4100 2700
+Wire Wire Line
+	4100 2700 4500 2700
+Wire Wire Line
+	3750 3000 3750 2900
+Wire Wire Line
+	4500 3000 3950 3000
+Wire Wire Line
+	3950 3000 3950 3250
+Wire Wire Line
+	3950 3550 3950 3650
 Wire Wire Line
 	5500 2500 5750 2500
@@
 P 3900 4700
 AR Path="/5E5B8164" Ref="C?"  Part="1"
-AR Path="/5E5A8A9D/5E5B8164" Ref="C?"  Part="1"
-F 0 "C?" H 4018 4746 50  0000 L CNN
+AR Path="/5E5A8A9D/5E5B8164" Ref="C2"  Part="1"
+F 0 "C2" H 4018 4746 50  0000 L CNN
 F 1 "10uF" H 4018 4655 50  0000 L CNN
-F 2 "" H 3938 4550 50  0001 C CNN
+F 2 "Capacitors:C_0603" H 3938 4550 50  0001 C CNN
 F 3 "~" H 3900 4700 50  0001 C CNN
 	1    3900 4700
@@
 P 4350 4700
 AR Path="/5E5B816A" Ref="C?"  Part="1"
-AR Path="/5E5A8A9D/5E5B816A" Ref="C?"  Part="1"
-F 0 "C?" H 4468 4746 50  0000 L CNN
+AR Path="/5E5A8A9D/5E5B816A" Ref="C3"  Part="1"
+F 0 "C3" H 4468 4746 50  0000 L CNN
 F 1 "0.1uF" H 4468 4655 50  0000 L CNN
-F 2 "" H 4388 4550 50  0001 C CNN
+F 2 "Capacitors:C_0603" H 4388 4550 50  0001 C CNN
 F 3 "~" H 4350 4700 50  0001 C CNN
 	1    4350 4700
@@
 P 5550 4700
 AR Path="/5E5B8170" Ref="C?"  Part="1"
-AR Path="/5E5A8A9D/5E5B8170" Ref="C?"  Part="1"
-F 0 "C?" H 5668 4746 50  0000 L CNN
+AR Path="/5E5A8A9D/5E5B8170" Ref="C4"  Part="1"
+F 0 "C4" H 5668 4746 50  0000 L CNN
 F 1 "0.1uF" H 5668 4655 50  0000 L CNN
-F 2 "" H 5588 4550 50  0001 C CNN
+F 2 "Capacitors:C_0603" H 5588 4550 50  0001 C CNN
 F 3 "~" H 5550 4700 50  0001 C CNN
 	1    5550 4700
@@
 P 6050 4700
 AR Path="/5E5B8176" Ref="C?"  Part="1"
-AR Path="/5E5A8A9D/5E5B8176" Ref="C?"  Part="1"
-F 0 "C?" H 6168 4746 50  0000 L CNN
+AR Path="/5E5A8A9D/5E5B8176" Ref="C6"  Part="1"
+F 0 "C6" H 6168 4746 50  0000 L CNN
 F 1 "10uF" H 6168 4655 50  0000 L CNN
-F 2 "" H 6088 4550 50  0001 C CNN
+F 2 "Capacitors:C_0603" H 6088 4550 50  0001 C CNN
 F 3 "~" H 6050 4700 50  0001 C CNN
 	1    6050 4700
@@
 P 4950 4500
 AR Path="/5E5B817C" Ref="U?"  Part="1"
-AR Path="/5E5A8A9D/5E5B817C" Ref="U?"  Part="1"
-F 0 "U?" H 4950 4742 50  0000 C CNN
+AR Path="/5E5A8A9D/5E5B817C" Ref="U1"  Part="1"
+F 0 "U1" H 4950 4742 50  0000 C CNN
 F 1 "AMS1117" H 4950 4651 50  0000 C CNN
 F 2 "Package_SOT:SOT-223" H 4950 4700 50  0001 C CNN
@@
 P 4950 4950
 AR Path="/5E5B8182" Ref="#PWR?"  Part="1"
-AR Path="/5E5A8A9D/5E5B8182" Ref="#PWR?"  Part="1"
-F 0 "#PWR?" H 4950 4700 50  0001 C CNN
+AR Path="/5E5A8A9D/5E5B8182" Ref="#PWR0107"  Part="1"
+F 0 "#PWR0107" H 4950 4700 50  0001 C CNN
 F 1 "GND" H 4950 4800 50  0001 C CNN
 F 2 "" H 4950 4950 50  0001 C CNN
@@
 Text GLabel 5600 2800 2    50   Input ~ 0
 ESP_RX
+Text GLabel 4450 2600 0    50   Input ~ 0
+Gas_A0
+Wire Wire Line
+	4450 2600 4500 2600
+Text GLabel 4400 3300 0    50   Input ~ 0
+SDA
+Text GLabel 4400 3200 0    50   Input ~ 0
+SCL
+Wire Wire Line
+	4400 3200 4500 3200
+Wire Wire Line
+	4400 3300 4500 3300
 $EndSCHEMATC

Commit message: pcb done
Connections:
- net Relay: now reaches U2.5 (GPIO14)
Changed lines of the file:
@@
 Wire Wire Line
 	4400 3300 4500 3300
+Text GLabel 4400 3100 0    50   Input ~ 0
+Relay
+Wire Wire Line
+	4500 3100 4400 3100
 $EndSCHEMATC
